File: TransverterBoard.kicad_pcb (KiCad board)
At the start: 2 copper layers, 44.4 x 65 mm, 27 parts, among them J1 Input Voltage, J2 RX Voltage, J3 TX Voltage, J4 IF, J5 RX, J6 TX, J7 VOX or Vin, K1 G5LE-1, K2 G5LE-1, Q1 TIP121

Commit message: working
Parts:
- added J8: Ext PTT, Connector_PinHeader_2.54mm:PinHeader_1x02_P2.54mm_Vertical, F.Cu at (27.9, 63.5)
- added R4: 2k2, Resistor_THT:R_Axial_DIN0207_L6.3mm_D2.5mm_P10.16mm_Horizontal, F.Cu at (43.8, 52.1)
- added U1: 4N25, Package_DIP:DIP-6_W7.62mm, F.Cu at (74.3, 85.1)
- moved C5 11.3 mm to (40.0, 46.4)
- moved L1 8.84 mm to (49.5, 47.1), turned to -90 degrees
- moved J2 5.08 mm to (38.1, 84.8)
- moved J3 5.08 mm to (38.1, 80.8)
- moved D3 4.04 mm to (41.3, 31.1)
- moved J1 3.36 mm to (34.3, 83.2)
- moved J4 3.05 mm to (34.9, 27.9)
- moved J7 2.79 mm to (41.1, 39.4)
- moved C2 2.79 mm to (40.9, 35.6)
- moved C3 1.99 mm to (52.0, 41.3)
- moved F1 0.76 mm to (36.8, 76.5)
- moved K1 0.62 mm to (43.6, 69.8)
Connections:
- L1 pad 1: Net-(D5-K) -> Net-(J7-Pin_3)
- L1 pad 2: Net-(J7-Pin_3) -> Net-(D5-K)
Routing:
- net Net-(J2-Pin_1): track 54.1 -> 0.00 mm
- net VOX_GND: track 89.9 -> 49.7 mm
- net +12V: track 82.3 -> 54.9 mm
- net Net-(J3-Pin_1): track 27.8 -> 4.93 mm
- net Net-(J1-Pin_2): track 9.43 -> 0.00 mm
- net Net-(D5-K): track 40.1 -> 30.8 mm
- net Net-(J7-Pin_3): track 6.96 -> 0.00 mm
- net Net-(D6-K): track 14.0 -> 7.76 mm
- net Net-(J7-Pin_1): track 4.10 -> 6.67 mm
- net Net-(J4-In): track 22.3 -> 23.9 mm
- net Net-(D4-K): track 13.5 -> 12.2 mm
- net Heat: vias 175 -> 0
- net (no net): vias 0 -> 175
- added copper zone on B.Cu, net (none)
- added copper zone on F.Cu, net (none)
- removed copper zone on B.Cu, net Heat
- removed copper zone on F.Cu, net Heat
