File: TransverterBoard.kicad_sch (KiCad schematic)
At the start: 27 parts, among them J1 Input Voltage, J2 RX Voltage, J3 TX Voltage, J4 IF, J5 RX, J6 TX, J7 VOX or Vin, K1 G5LE-1, K2 G5LE-1, Q1 TIP121

Commit message: Pcb
Parts:
- added HS1: Heatsink_Pad, Heatsink:Heatsink_35x26mm_1xFixation3mm_Fischer-SK486-35, symbol Mechanical:Heatsink_Pad
- C5: footprint (none) -> Capacitor_THT:CP_Radial_D6.3mm_P2.50mm
- D7: footprint (none) -> LED_THT:LED_D3.0mm_Clear
- J1: footprint (none) -> Connector_PinHeader_2.54mm:PinHeader_1x02_P2.54mm_Vertical
- Q1: footprint Package_TO_SOT_THT:TO-220-3_Vertical -> Package_TO_SOT_THT:TO-220-3_Horizontal_TabDown
- R1, R2, R3: footprint (none) -> Resistor_THT:R_Axial_DIN0207_L6.3mm_D2.5mm_P10.16mm_Horizontal
Connections:
- new net Heat: HS1.1
Changed lines of the file:
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@@
+    (stroke (width 0) (type default))
+  )
+  (wire (pts (xy 110.49 39.37) (xy 110.49 41.91))
     (stroke (width 0) (type default))
   )
@@
   )
   (wire (pts (xy 59.69 101.6) (xy 62.23 101.6))
+    (stroke (width 0) (type default))
+  )
+  (wire (pts (xy 106.68 41.91) (xy 110.49 41.91))
     (stroke (width 0) (type default))
   )
@@
     (property "Intersheetrefs" "${INTERSHEET_REFS}" (at 142.2619 30.48 0)
       (effects (font (size 1.27 1.27)) (justify left) hide)
+    )
+  )
+  (global_label "Heat" (shape input) (at 106.68 41.91 180) (fields_autoplaced)
+    (effects (font (size 1.27 1.27)) (justify right))
+    (property "Intersheetrefs" "${INTERSHEET_REFS}" (at 99.401 41.91 0)
+      (effects (font (size 1.27 1.27)) (justify right) hide)
     )
   )
@@
       (effects (font (size 1.27 1.27)) (justify left))
     )
-    (property "Footprint" "" (at 155.9052 77.47 0)
+    (property "Footprint" "Capacitor_THT:CP_Radial_D6.3mm_P2.50mm" (at 155.9052 77.47 0)
       (effects (font (size 1.27 1.27)) hide)
     )
@@
       (effects (font (size 1.27 1.27)) (justify left))
     )
-    (property "Footprint" "" (at 30.48 68.58 0)
+    (property "Footprint" "LED_THT:LED_D3.0mm_Clear" (at 30.48 68.58 0)
       (effects (font (size 1.27 1.27)) hide)
     )
@@
       (effects (font (size 1.27 1.27)))
     )
-    (property "Footprint" "" (at 45.72 33.02 0)
+    (property "Footprint" "Connector_PinHeader_2.54mm:PinHeader_1x02_P2.54mm_Vertical" (at 45.72 33.02 0)
       (effects (font (size 1.27 1.27)) hide)
     )
@@
       (effects (font (size 1.27 1.27)))
     )
-    (property "Footprint" "" (at 146.304 42.164 90)
+    (property "Footprint" "Resistor_THT:R_Axial_DIN0207_L6.3mm_D2.5mm_P10.16mm_Horizontal" (at 146.304 42.164 90)
       (effects (font (size 1.27 1.27)) hide)
     )
@@
     )
   )
+  (symbol (lib_id "Mechanical:Heatsink_Pad") (at 110.49 36.83 0) (unit 1)
+    (in_bom no) (on_board no) (dnp no) (fields_autoplaced)
+    (property "Reference" "HS1" (at 114.3 34.925 0)
+      (effects (font (size 1.27 1.27)) (justify left))
+    )
+    (property "Value" "Heatsink_Pad" (at 114.3 37.465 0)
+      (effects (font (size 1.27 1.27)) (justify left))
+    )
+    (property "Footprint" "Heatsink:Heatsink_35x26mm_1xFixation3mm_Fischer-SK486-35" (at 110.7948 38.1 0)
+      (effects (font (size 1.27 1.27)) hide)
+    )
+    (property "Datasheet" "~" (at 110.7948 38.1 0)
+      (effects (font (size 1.27 1.27)) hide)
+    )
+    (property "Sim.Enable" "0" (at 110.49 36.83 0)
+      (effects (font (size 1.27 1.27)) hide)
+    )
+    (pin "1")
+    (instances
+      (project "TransverterBoard"
+        (path "/7ff0e6ca-d973-406f-9317-cc62efc0df82"
+          (reference "HS1") (unit 1)
+        )
+      )
+    )
+  )
   (symbol (lib_id "Connector:Conn_01x03_Socket") (at 217.17 52.07 90) (unit 1)
     (in_bom yes) (on_board yes) (dnp no) (fields_autoplaced)
@@
       (effects (font (size 1.27 1.27)) (justify left))
     )
-    (property "Footprint" "Package_TO_SOT_THT:TO-220-3_Vertical" (at 125.73 45.085 0)
+    (property "Footprint" "Package_TO_SOT_THT:TO-220-3_Horizontal_TabDown" (at 125.73 45.085 0)
       (effects (font (size 1.27 1.27) italic) (justify left) hide)
     )
@@
       (effects (font (size 1.27 1.27)) (justify left))
     )
-    (property "Footprint" "" (at 155.956 52.324 90)
+    (property "Footprint" "Resistor_THT:R_Axial_DIN0207_L6.3mm_D2.5mm_P10.16mm_Horizontal" (at 155.956 52.324 90)
       (effects (font (size 1.27 1.27)) hide)
     )
@@
       (effects (font (size 1.27 1.27)) (justify left))
     )
-    (property "Footprint" "" (at 31.496 58.674 90)
-      (effects (font (size 1.27 1.27)) hide)
-    )
+    (property "Footprint" "Resistor_THT:R_Axial_DIN0207_L6.3mm_D2.5mm_P10.16mm_Horizontal" (at 31.496 58.674 90)
+      (effects (font (size 1.27 1.27)) hide)
+    )

Commit message: working
Parts:
- added J8: Ext PTT, Connector_PinHeader_2.54mm:PinHeader_1x02_P2.54mm_Vertical, symbol Connector:Conn_01x02_Socket
- added R4: 2k2, Resistor_THT:R_Axial_DIN0207_L6.3mm_D2.5mm_P10.16mm_Horizontal, symbol Device:R_US
- added U1: 4N25, Package_DIP:DIP-6_W7.62mm, symbol Isolator:4N25
Connections:
- net +12V: now also R4.2
- net GND: now also J8.2 (Pin_2), U1.5
- net VOX_GND: now also U1.4
- net at C4.2, D5.1 (K), D6.2 (A)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: now also L1.2; no longer L1.1
- net at J7.3 (Pin_3): now also L1.1; no longer L1.2
- new net: J8.1 (Pin_1), U1.1
- new net: R4.1, U1.2
Other:
- moved on the sheet: L1
Changed lines of the file:
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@@
+    (stroke (width 0) (type default))
+  )
+  (wire (pts (xy 140.97 101.6) (xy 144.78 101.6))
     (stroke (width 0) (type default))
   )
@@
     (stroke (width 0) (type default))
   )
+  (wire (pts (xy 171.45 109.22) (xy 171.45 110.49))
+    (stroke (width 0) (type default))
+  )
   (wire (pts (xy 149.86 43.18) (xy 154.94 43.18))
     (stroke (width 0) (type default))
@@
     (stroke (width 0) (type default))
   )
+  (wire (pts (xy 160.02 101.6) (xy 162.56 101.6))
+    (stroke (width 0) (type default))
+  )
   (wire (pts (xy 67.31 109.22) (xy 69.85 109.22))
     (stroke (width 0) (type default))
   )
+  (wire (pts (xy 170.18 101.6) (xy 173.99 101.6))
+    (stroke (width 0) (type default))
+  )
+  (wire (pts (xy 173.99 109.22) (xy 171.45 109.22))
+    (stroke (width 0) (type default))
+  )
   (wire (pts (xy 67.31 96.52) (xy 69.85 96.52))
     (stroke (width 0) (type default))
@@
     (stroke (width 0) (type default))
   )
+  (wire (pts (xy 139.7 104.14) (xy 139.7 107.95))
+    (stroke (width 0) (type default))
+  )
   (wire (pts (xy 74.93 63.5) (xy 64.77 63.5))
     (stroke (width 0) (type default))
@@
     (stroke (width 0) (type default))
   )
+  (wire (pts (xy 139.7 104.14) (xy 144.78 104.14))
+    (stroke (width 0) (type default))
+  )
   (wire (pts (xy 59.69 114.3) (xy 62.23 114.3))
     (stroke (width 0) (type default))
   )
+  (wire (pts (xy 173.99 101.6) (xy 173.99 97.79))
+    (stroke (width 0) (type default))
+  )
   (wire (pts (xy 67.31 91.44) (xy 69.85 91.44))
+    (stroke (width 0) (type default))
+  )
+  (wire (pts (xy 160.02 106.68) (xy 173.99 106.68))
     (stroke (width 0) (type default))
   )
@@
     (property "Intersheetrefs" "${INTERSHEET_REFS}" (at 99.401 41.91 0)
       (effects (font (size 1.27 1.27)) (justify right) hide)
+    )
+  )
+  (global_label "VOX_GND" (shape input) (at 140.97 101.6 180) (fields_autoplaced)
+    (effects (font (size 1.27 1.27)) (justify right))
+    (property "Intersheetrefs" "${INTERSHEET_REFS}" (at 129.5181 101.6 0)
+      (effects (font (size 1.27 1.27)) (justify right) hide)
+    )
+  )
+  (symbol (lib_id "Connector:Conn_01x02_Socket") (at 179.07 106.68 0) (unit 1)
+    (in_bom yes) (on_board yes) (dnp no) (fields_autoplaced)
+    (property "Reference" "J8" (at 180.34 106.68 0)
+      (effects (font (size 1.27 1.27)) (justify left))
+    )
+    (property "Value" "Ext PTT" (at 180.34 109.22 0)
+      (effects (font (size 1.27 1.27)) (justify left))
+    )
+    (property "Footprint" "Connector_PinHeader_2.54mm:PinHeader_1x02_P2.54mm_Vertical" (at 179.07 106.68 0)
+      (effects (font (size 1.27 1.27)) hide)
+    )
+    (property "Datasheet" "~" (at 179.07 106.68 0)
+      (effects (font (size 1.27 1.27)) hide)
+    )
+    (pin "1")
+    (pin "2")
+    (instances
+      (project "TransverterBoard"
+        (path "/7ff0e6ca-d973-406f-9317-cc62efc0df82"
+          (reference "J8") (unit 1)
+        )
+      )
     )
   )
@@
     )
   )
-  (symbol (lib_id "Device:L") (at 181.61 43.18 90) (unit 1)
+  (symbol (lib_id "Device:L") (at 181.61 43.18 270) (unit 1)
     (in_bom yes) (on_board yes) (dnp no) (fields_autoplaced)
     (property "Reference" "L1" (at 181.61 38.1 90)
@@
     )
   )
+  (symbol (lib_id "power:+12V") (at 173.99 97.79 0) (unit 1)
+    (in_bom yes) (on_board yes) (dnp no) (fields_autoplaced)
+    (property "Reference" "#PWR012" (at 173.99 101.6 0)
+      (effects (font (size 1.27 1.27)) hide)
+    )
+    (property "Value" "+12V" (at 173.99 92.71 0)
+      (effects (font (size 1.27 1.27)))
+    )
+    (property "Footprint" "" (at 173.99 97.79 0)
+      (effects (font (size 1.27 1.27)) hide)
+    )
+    (property "Datasheet" "" (at 173.99 97.79 0)
+      (effects (font (size 1.27 1.27)) hide)
+    )
+    (pin "1")
+    (instances
+      (project "TransverterBoard"
+        (path "/7ff0e6ca-d973-406f-9317-cc62efc0df82"
+          (reference "#PWR012") (unit 1)
+        )
+      )
+    )
+  )
   (symbol (lib_id "Relay:G5LE-1") (at 237.49 72.39 180) (unit 1)
     (in_bom yes) (on_board yes) (dnp no) (fields_autoplaced)
@@
     )
   )
+  (symbol (lib_id "Isolator:4N25") (at 152.4 104.14 180) (unit 1)
+    (in_bom yes) (on_board yes) (dnp no) (fields_autoplaced)
+    (property "Reference" "U1" (at 152.4 95.25 0)
+      (effects (font (size 1.27 1.27)))
+    )
+    (property "Value" "4N25" (at 152.4 97.79 0)
+      (effects (font (size 1.27 1.27)))
+    )
+    (property "Footprint" "Package_DIP:DIP-6_W7.62mm" (at 157.48 99.06 0)
+      (effects (font (size 1.27 1.27) italic) (justify left) hide)
+    )
+    (property "Datasheet" "https://www.vishay.com/docs/83725/4n25.pdf" (at 152.4 104.14 0)
+      (effects (font (size 1.27 1.27)) (justify left) hide)
+    )
+    (pin "1")
+    (pin "2")
+    (pin "3")
+    (pin "4")
+    (pin "5")
+    (pin "6")
+    (instances
+      (project "TransverterBoard"
+        (path "/7ff0e6ca-d973-406f-9317-cc62efc0df82"
+          (reference "U1") (unit 1)
+        )
+      )
+    )
+  )
   (symbol (lib_id "Mechanical:Heatsink_Pad") (at 110.49 36.83 0) (unit 1)
     (in_bom no) (on_board no) (dnp no) (fields_autoplaced)
@@
     )
   )
+  (symbol (lib_id "Device:R_US") (at 166.37 101.6 90) (unit 1)
+    (in_bom yes) (on_board yes) (dnp no) (fields_autoplaced)
+    (property "Reference" "R4" (at 166.37 95.25 90)
+      (effects (font (size 1.27 1.27)))
+    )
+    (property "Value" "2k2" (at 166.37 97.79 90)
+      (effects (font (size 1.27 1.27)))
+    )
+    (property "Footprint" "Resistor_THT:R_Axial_DIN0207_L6.3mm_D2.5mm_P10.16mm_Horizontal" (at 166.624 100.584 90)
+      (effects (font (size 1.27 1.27)) hide)
+    )
+    (property "Datasheet" "~" (at 166.37 101.6 0)
+      (effects (font (size 1.27 1.27)) hide)
+    )
+    (pin "1")
+    (pin "2")
+    (instances
+      (project "TransverterBoard"
+        (path "/7ff0e6ca-d973-406f-9317-cc62efc0df82"
+          (reference "R4") (unit 1)
+        )
+      )
+    )
+  )
   (symbol (lib_id "Relay:G5LE-1") (at 69.85 73.66 180) (unit 1)
     (in_bom yes) (on_board yes) (dnp no) (fields_autoplaced)
@@
         )
       )
+    )
+  )
+  (symbol (lib_id "power:GND") (at 171.45 110.49 0) (unit 1)
+    (in_bom yes) (on_board yes) (dnp no) (fields_autoplaced)
+    (property "Reference" "#PWR013" (at 171.45 116.84 0)
+      (effects (font (size 1.27 1.27)) hide)
+    )
+    (property "Value" "GND" (at 171.45 115.57 0)
+      (effects (font (size 1.27 1.27)))
+    )
+    (property "Footprint" "" (at 171.45 110.49 0)
+      (effects (font (size 1.27 1.27)) hide)
+    )
+    (property "Datasheet" "" (at 171.45 110.49 0)
+      (effects (font (size 1.27 1.27)) hide)
+    )
+    (pin "1")
+    (instances
+      (project "TransverterBoard"
+        (path "/7ff0e6ca-d973-406f-9317-cc62efc0df82"
+          (reference "#PWR013") (unit 1)
+        )
+      )
+    )
+  )
+  (symbol (lib_id "power:GND") (at 139.7 107.95 0) (unit 1)
+    (in_bom yes) (on_board yes) (dnp no) (fields_autoplaced)
+    (property "Reference" "#PWR011" (at 139.7 114.3 0)
+      (effects (font (size 1.27 1.27)) hide)
+    )
+    (property "Value" "GND" (at 139.7 113.03 0)
+      (effects (font (size 1.27 1.27)))
+    )
+    (property "Footprint" "" (at 139.7 107.95 0)
+      (effects (font (size 1.27 1.27)) hide)
+    )
+    (property "Datasheet" "" (at 139.7 107.95 0)
+      (effects (font (size 1.27 1.27)) hide)
+    )
+    (pin "1")
+    (instances
+      (project "TransverterBoard"
+        (path "/7ff0e6ca-d973-406f-9317-cc62efc0df82"
+          (reference "#PWR011") (unit 1)
+        )
+      )
